File: Keystrip_detachable/KeyStrip.kicad_sch (KiCad schematic)
At the start: 13 parts, among them J1 JST_06, J2 JST_08, J3 JST_06, J4 JST_06

Commit message: ah
Parts:
- removed J2: JST_08, Library:JST_EH_B8B-EH-A_1x08_P2.50mm_Vertical, symbol PCM_SL_Connectors:JST_08
- removed J4: JST_06, Library:6pin, symbol PCM_SL_Connectors:JST_06
- added J4: JST_08, Library:JST_EH_B8B-EH-A_1x08_P2.50mm_Vertical, symbol PCM_SL_Connectors:JST_08
Connections:
- net 2: now reaches D7.1 (K), J1.6
- net 2: now also J4.2
- net 4: now reaches J1.1, J3.1, S4.1, S5.1, S6.1
- net 4: now also J4.4
- net 1: now reaches D9.1 (K)
- net 1: now also J4.1
- net 3: now reaches D8.1 (K), J3.6
- net 3: now also J4.3
- net 5: now reaches D12.2 (DOUT)
- net 5: now also J4.5
- net 6: now reaches D10.1 (VDD), D11.1 (VDD), D12.1 (VDD), J1.4, J3.4
- net 6: now also J4.6
- net 7: now reaches D10.4 (DIN), J1.3
- net 7: now also J4.7
- net 8: now reaches D10.3 (VSS), D11.3 (VSS), D12.3 (VSS), J1.2, J3.2
- net 8: now also J4.8

Commit message: uhhh, This feels both improved and weirder
Connections:
- net 6: now also J1.5; no longer J1.4
- net 7: now also J1.2; no longer J1.3
- net 8: now also J1.3; no longer J1.2
- net at D10.2 (DOUT), D11.4 (DIN), J3.3: now also J1.4; no longer J1.5
Changed lines of the file:
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@@
+	)
+	(junction
+		(at 115.57 80.01)
+		(diameter 0)
+		(color 0 0 0 0)
 	)
 	(junction
@@
 	)
 	(junction
+		(at 152.4 102.87)
+		(diameter 0)
+		(color 0 0 0 0)
+	)
+	(junction
+		(at 137.16 102.87)
+		(diameter 0)
+		(color 0 0 0 0)
+	)
+	(junction
+		(at 137.16 66.04)
+		(diameter 0)
+		(color 0 0 0 0)
+	)
+	(junction
+		(at 152.4 72.39)
+		(diameter 0)
+		(color 0 0 0 0)
+	)
+	(junction
+		(at 144.78 95.25)
+		(diameter 0)
+		(color 0 0 0 0)
+	)
+	(junction
 		(at 144.78 73.66)
 		(diameter 0)
@@
 	)
 	(junction
-		(at 152.4 102.87)
-		(diameter 0)
-		(color 0 0 0 0)
-	)
-	(junction
-		(at 152.4 71.12)
-		(diameter 0)
-		(color 0 0 0 0)
-	)
-	(junction
-		(at 137.16 102.87)
-		(diameter 0)
-		(color 0 0 0 0)
-	)
-	(junction
-		(at 137.16 66.04)
-		(diameter 0)
-		(color 0 0 0 0)
-	)
-	(junction
-		(at 144.78 95.25)
-		(diameter 0)
-		(color 0 0 0 0)
-	)
-	(junction
 		(at 127 92.71)
 		(diameter 0)
@@
 	(wire
 		(pts
-			(xy 115.57 78.74) (xy 115.57 95.25)
+			(xy 115.57 78.74) (xy 115.57 80.01)
 		)
 		(stroke
@@
 	(wire
 		(pts
+			(xy 144.78 69.85) (xy 144.78 73.66)
+		)
+		(stroke
+			(width 0)
+			(type default)
+		)
+	)
+	(wire
+		(pts
 			(xy 152.4 83.82) (xy 152.4 90.17)
 		)
@@
 	(wire
 		(pts
+			(xy 152.4 72.39) (xy 152.4 83.82)
+		)
+		(stroke
+			(width 0)
+			(type default)
+		)
+	)
+	(wire
+		(pts
+			(xy 153.67 58.42) (xy 153.67 59.69)
+		)
+		(stroke
+			(width 0)
+			(type default)
+		)
+	)
+	(wire
+		(pts
 			(xy 137.16 102.87) (xy 137.16 114.3)
 		)
@@
 	(wire
 		(pts
-			(xy 153.67 67.31) (xy 165.1 67.31)
-		)
-		(stroke
-			(width 0)
-			(type default)
-		)
-	)
-	(wire
-		(pts
 			(xy 163.83 87.63) (xy 165.1 87.63)
 		)
@@
 	(wire
 		(pts
-			(xy 153.67 59.69) (xy 153.67 67.31)
-		)
-		(stroke
-			(width 0)
-			(type default)
-		)
-	)
-	(wire
-		(pts
 			(xy 115.57 62.23) (xy 115.57 78.74)
 		)
@@
 	(wire
 		(pts
-			(xy 154.94 57.15) (xy 137.16 57.15)
-		)
-		(stroke
-			(width 0)
-			(type default)
-		)
-	)
-	(wire
-		(pts
-			(xy 152.4 71.12) (xy 165.1 71.12)
-		)
-		(stroke
-			(width 0)
-			(type default)
-		)
-	)
-	(wire
-		(pts
 			(xy 152.4 90.17) (xy 152.4 102.87)
 		)
@@
 	(wire
 		(pts
-			(xy 165.1 78.74) (xy 165.1 80.01)
-		)
-		(stroke
-			(width 0)
-			(type default)
-		)
-	)
-	(wire
-		(pts
 			(xy 132.08 96.52) (xy 165.1 96.52)
 		)
@@
 	(wire
 		(pts
-			(xy 165.1 64.77) (xy 154.94 64.77)
-		)
-		(stroke
-			(width 0)
-			(type default)
-		)
-	)
-	(wire
-		(pts
 			(xy 127 91.44) (xy 127 92.71)
 		)
@@
 	(wire
 		(pts
-			(xy 152.4 71.12) (xy 152.4 83.82)
-		)
-		(stroke
-			(width 0)
-			(type default)
-		)
-	)
-	(wire
-		(pts
 			(xy 156.21 77.47) (xy 156.21 82.55)
 		)
@@
 	(wire
 		(pts
+			(xy 144.78 73.66) (xy 144.78 76.2)
+		)
+		(stroke
+			(width 0)
+			(type default)
+		)
+	)
+	(wire
+		(pts
 			(xy 153.67 95.25) (xy 144.78 95.25)
 		)
@@
 	(wire
 		(pts
+			(xy 154.94 67.31) (xy 165.1 67.31)
+		)
+		(stroke
+			(width 0)
+			(type default)
+		)
+	)
+	(wire
+		(pts
+			(xy 137.16 57.15) (xy 154.94 57.15)
+		)
+		(stroke
+			(width 0)
+			(type default)
+		)
+	)
+	(wire
+		(pts
+			(xy 152.4 72.39) (xy 165.1 72.39)
+		)
+		(stroke
+			(width 0)
+			(type default)
+		)
+	)
+	(wire
+		(pts
 			(xy 135.89 57.15) (xy 135.89 55.88)
 		)
@@
 	(wire
 		(pts
+			(xy 144.78 69.85) (xy 165.1 69.85)
+		)
+		(stroke
+			(width 0)
+			(type default)
+		)
+	)
+	(wire
+		(pts
 			(xy 144.78 109.22) (xy 144.78 110.49)
 		)
@@
 	(wire
 		(pts
-			(xy 165.1 71.12) (xy 165.1 69.85)
-		)
-		(stroke
-			(width 0)
-			(type default)
-		)
-	)
-	(wire
-		(pts
-			(xy 154.94 64.77) (xy 154.94 57.15)
+			(xy 154.94 57.15) (xy 154.94 67.31)
 		)
 		(stroke
@@
 	(wire
 		(pts
-			(xy 153.67 59.69) (xy 153.67 58.42)
-		)
-		(stroke
-			(width 0)
-			(type default)
-		)
-	)
-	(wire
-		(pts
 			(xy 165.1 91.44) (xy 165.1 90.17)
 		)
@@
 	(wire
 		(pts
-			(xy 144.78 73.66) (xy 165.1 73.66)
-		)
-		(stroke
-			(width 0)
-			(type default)
-		)
-	)
-	(wire
-		(pts
 			(xy 120.65 74.93) (xy 132.08 74.93)
 		)
@@
 	(wire
 		(pts
-			(xy 115.57 78.74) (xy 165.1 78.74)
+			(xy 115.57 80.01) (xy 165.1 80.01)
 		)
 		(stroke
@@
 	(wire
 		(pts
+			(xy 153.67 64.77) (xy 165.1 64.77)
+		)
+		(stroke
+			(width 0)
+			(type default)
+		)
+	)
+	(wire
+		(pts
 			(xy 132.08 74.93) (xy 165.1 74.93)
 		)
@@
 	(wire
 		(pts
-			(xy 144.78 73.66) (xy 144.78 76.2)
-		)
-		(stroke
-			(width 0)
-			(type default)
-		)
-	)
-	(wire
-		(pts
-			(xy 152.4 66.04) (xy 152.4 71.12)
+			(xy 152.4 66.04) (xy 152.4 72.39)
 		)
 		(stroke
@@
 	(wire
 		(pts
-			(xy 165.1 73.66) (xy 165.1 72.39)
+			(xy 153.67 59.69) (xy 153.67 64.77)
 		)
 		(stroke
@@
 		)
 		(stroke
+			(width 0)
+			(type default)
+		)
+	)
+	(wire
+		(pts
+			(xy 115.57 80.01) (xy 115.57 95.25)
+		)
+		(stroke

Commit message: still artistic... Cleaner IG?
Connections:
- net 1: now also J4.2; no longer J4.1
- net 2: now also J4.1; no longer J4.2
- net 3: now also J4.7; no longer J4.3
- net 4: now also J4.6; no longer J4.4
- net 5: now also J4.4; no longer J4.5
- net 6: now also J3.5, J4.3; no longer J3.4, J4.6
- net 7: now also J4.8; no longer J4.7
- net 8: now also J3.3, J4.5; no longer J3.2, J4.8
- net at D10.2 (DOUT), D11.4 (DIN), J1.4: now also J3.2; no longer J3.3
- net at D11.2 (DOUT), D12.4 (DIN): now also J3.4; no longer J3.5
Changed lines of the file:
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@@
+	)
+	(junction
+		(at 144.78 91.44)
+		(diameter 0)
+		(color 0 0 0 0)
 	)
 	(junction
@@
 	)
 	(junction
-		(at 144.78 91.44)
-		(diameter 0)
-		(color 0 0 0 0)
-	)
-	(junction
 		(at 115.57 95.25)
 		(diameter 0)
@@
 	(wire
 		(pts
-			(xy 163.83 90.17) (xy 163.83 87.63)
-		)
-		(stroke
-			(width 0)
-			(type default)
-		)
-	)
-	(wire
-		(pts
 			(xy 115.57 78.74) (xy 115.57 80.01)
 		)
@@
 	(wire
 		(pts
-			(xy 144.78 91.44) (xy 165.1 91.44)
-		)
-		(stroke
-			(width 0)
-			(type default)
-		)
-	)
-	(wire
-		(pts
 			(xy 165.1 104.14) (xy 153.67 104.14)
 		)
@@
 	(wire
 		(pts
-			(xy 163.83 87.63) (xy 165.1 87.63)
-		)
-		(stroke
-			(width 0)
-			(type default)
-		)
-	)
-	(wire
-		(pts
 			(xy 115.57 62.23) (xy 115.57 78.74)
 		)
@@
 	(wire
 		(pts
-			(xy 165.1 85.09) (xy 153.67 85.09)
-		)
-		(stroke
-			(width 0)
-			(type default)
-		)
-	)
-	(wire
-		(pts
 			(xy 127 91.44) (xy 127 92.71)
 		)
@@
 	(wire
 		(pts
-			(xy 156.21 77.47) (xy 156.21 82.55)
-		)
-		(stroke
-			(width 0)
-			(type default)
-		)
-	)
-	(wire
-		(pts
 			(xy 127 92.71) (xy 127 116.84)
 		)
@@
 	(wire
 		(pts
+			(xy 144.78 91.44) (xy 148.59 91.44)
+		)
+		(stroke
+			(width 0)
+			(type default)
+		)
+	)
+	(wire
+		(pts
 			(xy 115.57 95.25) (xy 115.57 99.06)
 		)
@@
 	(wire
 		(pts
+			(xy 148.59 87.63) (xy 165.1 87.63)
+		)
+		(stroke
+			(width 0)
+			(type default)
+		)
+	)
+	(wire
+		(pts
 			(xy 153.67 95.25) (xy 144.78 95.25)
 		)
@@
 	(wire
 		(pts
+			(xy 144.78 91.44) (xy 144.78 95.25)
+		)
+		(stroke
+			(width 0)
+			(type default)
+		)
+	)
+	(wire
+		(pts
 			(xy 137.16 57.15) (xy 154.94 57.15)
 		)
@@
 	(wire
 		(pts
-			(xy 144.78 91.44) (xy 144.78 95.25)
-		)
-		(stroke
-			(width 0)
-			(type default)
-		)
-	)
-	(wire
-		(pts
 			(xy 137.16 114.3) (xy 166.37 114.3)
 		)
@@
 	(wire
 		(pts
-			(xy 165.1 91.44) (xy 165.1 90.17)
+			(xy 148.59 91.44) (xy 148.59 87.63)
 		)
 		(stroke
@@
 	(wire
 		(pts
-			(xy 156.21 82.55) (xy 165.1 82.55)
+			(xy 153.67 82.55) (xy 165.1 82.55)
 		)
 		(stroke
@@
 	(wire
 		(pts
+			(xy 153.67 76.2) (xy 153.67 82.55)
+		)
+		(stroke
+			(width 0)
+			(type default)
+		)
+	)
+	(wire
+		(pts
 			(xy 137.16 57.15) (xy 137.16 66.04)
 		)
@@
 	(wire
 		(pts
-			(xy 152.4 90.17) (xy 163.83 90.17)
+			(xy 156.21 85.09) (xy 165.1 85.09)
+		)
+		(stroke
+			(width 0)
+			(type default)
+		)
+	)
+	(wire
+		(pts
+			(xy 152.4 90.17) (xy 165.1 90.17)
 		)
 		(stroke
@@
 	(wire
 		(pts
+			(xy 156.21 77.47) (xy 156.21 85.09)
+		)
+		(stroke
+			(width 0)
+			(type default)
+		)
+	)
+	(wire
+		(pts
 			(xy 115.57 57.15) (xy 135.89 57.15)
 		)
@@
 	(wire
 		(pts
-			(xy 153.67 85.09) (xy 153.67 76.2)
-		)
-		(stroke
-			(width 0)
-			(type default)
-		)
-	)
-	(wire
-		(pts
 			(xy 115.57 80.01) (xy 115.57 95.25)
 		)
@@
 			(width 0)
 			(type default)
-		)
-	)
-	(label "6"
-		(at 175.26 114.3 0)
-		(effects
-			(font
-				(size 1.27 1.27)
-			)
-			(justify left bottom)
 		)
 	)
@@
 		)
 	)
-	(label "1"
-		(at 175.26 101.6 0)
-		(effects
-			(font
-				(size 1.27 1.27)
-			)
-			(justify left bottom)
-		)
-	)
 	(label "5"
-		(at 175.26 111.76 0)
-		(effects
-			(font
-				(size 1.27 1.27)
-			)
-			(justify left bottom)
-		)
-	)
-	(label "8"
-		(at 175.26 119.38 0)
+		(at 175.26 109.22 0)
+		(effects
+			(font
+				(size 1.27 1.27)
+			)
+			(justify left bottom)
+		)
+	)
+	(label "4"
+		(at 175.26 114.3 0)
+		(effects
+			(font
+				(size 1.27 1.27)
+			)
+			(justify left bottom)
+		)
+	)
+	(label "6"
+		(at 175.26 106.68 0)
 		(effects
 			(font
@@
 		)
 	)
-	(label "3"
-		(at 175.26 106.68 0)
+	(label "1"
+		(at 175.26 104.14 0)
 		(effects
 			(font
@@
 		)
 	)
-	(label "4"
-		(at 175.26 109.22 0)
+	(label "2"
+		(at 175.26 101.6 0)
+		(effects
+			(font
+				(size 1.27 1.27)
+			)
+			(justify left bottom)
+		)
+	)
+	(label "7"
+		(at 175.26 119.38 0)
 		(effects
 			(font
@@
 		)
 	)
+	(label "3"
+		(at 175.26 116.84 0)
+		(effects
+			(font
+				(size 1.27 1.27)
+			)
+			(justify left bottom)
+		)
+	)
+	(label "8"
+		(at 175.26 111.76 0)
+		(effects
+			(font
+				(size 1.27 1.27)
+			)
+			(justify left bottom)
+		)
+	)
 	(label "1"
 		(at 165.1 111.76 0)
@@
 		)
 	)
-	(label "7"
-		(at 175.26 116.84 0)
-		(effects
-			(font
-				(size 1.27 1.27)
-			)
-			(justify left bottom)
-		)
-	)
 	(label "3"
 		(at 166.37 116.84 0)
 		(effects
 			(font
-				(size 1.27 1.27)
-			)
-			(justify left bottom)
-		)
-	)
-	(label "2"
-		(at 175.26 104.14 0)
-		(effects
-			(font
