File: Keystrip_detachable/KeyStrip.kicad_pcb (KiCad board)
At the start: 2 copper layers, 19.1 x 57.2 mm, 13 parts, among them J1 JST_06, J2 JST_08, J3 JST_06, J4 JST_06

Commit message: ah
Parts:
- added J4: JST_08, Library:JST_EH_B8B-EH-A_1x08_P2.50mm_Vertical, F.Cu at (95.0, 115.5)
- added REF**: MouseBite-Slot_2.0x2.0mm_outset_D0.5mm_P0.85mm_2h_Trace, Panelization:MouseBite-Slot_2.0x2.0mm_outset_D0.5mm_P0.85mm_2h_Trace, F.Cu at (61.8, 114.8)
- added REF**: LilHole, Library:LilHole, F.Cu at (76.8, 97.8)
- added REF**: LilHole, Library:LilHole, F.Cu at (65.8, 97.8)
- added REF**: LilHole, Library:LilHole, F.Cu at (76.8, 78.7)
- added REF**: LilHole, Library:LilHole, F.Cu at (65.8, 78.7)
Connections:
- D10 pad 1: Net-(D10-VDD) -> /6
- D10 pad 3: Net-(D10-VSS) -> /8
- D10 pad 4: Net-(D10-DIN) -> /7
- D11 pad 1: Net-(D10-VDD) -> /6
- D11 pad 3: Net-(D10-VSS) -> /8
- D12 pad 1: Net-(D10-VDD) -> /6
- D12 pad 2: Net-(D12-DOUT) -> /5
- D12 pad 3: Net-(D10-VSS) -> /8
- D7 pad 1: Net-(D7-K) -> /2
- D8 pad 1: Net-(D8-K) -> /3
- D9 pad 1: Net-(D9-K) -> /1
- J1 pad 1: Net-(J1-Pad1) -> /4
- J1 pad 2: Net-(D10-VSS) -> /8
- J1 pad 3: Net-(D10-DIN) -> /7
- J1 pad 4: Net-(D10-VDD) -> /6
- J1 pad 6: Net-(D7-K) -> /2
- J3 pad 1: Net-(J1-Pad1) -> /4
- J3 pad 2: Net-(D10-VSS) -> /8
- J3 pad 4: Net-(D10-VDD) -> /6
- J3 pad 6: Net-(D8-K) -> /3
- S4 pad 1: Net-(J1-Pad1) -> /4
- S5 pad 1: Net-(J1-Pad1) -> /4
- S6 pad 1: Net-(J1-Pad1) -> /4

Commit message: uhhh, This feels both improved and weirder
Parts:
- removed J2: JST_08, Library:JST_EH_B8B-EH-A_1x08_P2.50mm_Vertical
- removed the J4 at (62.8, 102.5)
- removed the REF** at (61.8, 114.8)
- removed the REF** at (76.8, 97.8)
- removed the REF** at (65.8, 97.8)
- removed the REF** at (76.8, 78.7)
- removed the REF** at (65.8, 78.7)
- added ?: , , F.Cu at (77.6, 80.5)
- added ?: , , F.Cu at (63.2, 80.5)
- added ?: , , F.Cu at (63.2, 99.5)
- added ?: , , F.Cu at (64.9, 99.5)
- added ?: , , F.Cu at (79.3, 99.5)
- added ?: , , F.Cu at (64.9, 98.0)
- added ?: , , F.Cu at (79.3, 80.5)
- added ?: , , F.Cu at (64.9, 79.0)
- added ?: , , F.Cu at (64.9, 80.5)
- added ?: , , F.Cu at (77.6, 98.0)
- added ?: , , F.Cu at (77.6, 79.0)
- added REF**: LilHole, Library:LilHole, F.Cu at (77.6, 99.5)
- moved J4 30.8 mm to (64.2, 115.7)
- moved J1 18.9 mm to (76.2, 77.5), turned to 180 degrees
- moved J3 18.8 mm to (76.2, 96.5), turned to 180 degrees
Connections:
- J1 pad 2: /8 -> /7
- J1 pad 3: /7 -> /8
- J1 pad 4: /6 -> Net-(D10-DOUT)
- J1 pad 5: Net-(D10-DOUT) -> /6
Routing:
- net Net-(D10-VSS): track 102.0 -> 0.00 mm, vias 4 -> 0
- net Net-(J1-Pad1): track 98.8 -> 0.00 mm, vias 1 -> 0
- net Net-(D10-VDD): track 87.6 -> 0.00 mm, vias 9 -> 0
- net Net-(D10-DIN): track 73.9 -> 0.00 mm, vias 4 -> 0
- net Net-(D7-K): track 71.3 -> 0.00 mm, vias 2 -> 0
- net Net-(D8-K): track 52.3 -> 0.00 mm, vias 1 -> 0
- net Net-(D11-DOUT): track 39.9 -> 0.00 mm, vias 4 -> 0
- net Net-(D9-K): track 39.1 -> 0.00 mm, vias 4 -> 0
- net Net-(D10-DOUT): track 37.0 -> 0.00 mm, vias 4 -> 0
- net Net-(D12-DOUT): track 11.3 -> 0.00 mm, vias 2 -> 0
- net /3: track 0.00 -> 2.14 mm
- net /2: track 0.00 -> 2.14 mm
- net /1: track 0.00 -> 2.14 mm
- net /7: track 0.00 -> 0.85 mm
Other:
- outline, holes or cut-outs redrawn
- board text removed: "${REFERENCE}"

Commit message: still artistic... Cleaner IG?
Parts:
- moved D7 0.41 mm to (79.8, 73.0)
- moved D9 0.26 mm to (79.8, 111.1)
- moved D8 0.22 mm to (79.8, 92.0)
Connections:
- J3 pad 2: /8 -> Net-(D10-DOUT)
- J3 pad 3: Net-(D10-DOUT) -> /8
- J3 pad 4: /6 -> Net-(D11-DOUT)
- J3 pad 5: Net-(D11-DOUT) -> /6
- J4 pad 1: /1 -> /2
- J4 pad 2: /2 -> /1
- J4 pad 3: /3 -> /6
- J4 pad 4: /4 -> /5
- J4 pad 5: /5 -> /8
- J4 pad 6: /6 -> /4
- J4 pad 7: /7 -> /3
- J4 pad 8: /8 -> /7
Routing:
- net /4: track 0.00 -> 75.2 mm
- net /2: track 2.14 -> 63.0 mm, vias 0 -> 1
- net /8: track 0.00 -> 58.7 mm, vias 0 -> 3
- net /6: track 0.00 -> 56.7 mm, vias 0 -> 5
- net /3: track 2.14 -> 53.5 mm, vias 0 -> 3
- net /7: track 0.85 -> 52.1 mm, vias 0 -> 3
- net Net-(D10-DOUT): track 0.00 -> 37.0 mm, vias 0 -> 2
- net Net-(D11-DOUT): track 0.00 -> 31.3 mm, vias 0 -> 2
- net /1: track 2.14 -> 22.6 mm, vias 0 -> 1
- net /5: track 0.00 -> 3.36 mm

Commit message: uhh
Parts:
- added REF**: EC11_Switch, reversible-kicad-footprints:EC11_Switch, F.Cu at (71.2, 69.2)
- added REF**: RJ45_Ninigi_GE, Connector_RJ:RJ45_Ninigi_GE, F.Cu at (66.1, 64.1)
